File: hw/v1/v1.kicad_pcb (KiCad board)
At the start: 2 copper layers, 44.9 x 29.9 mm, 35 parts, among them J1 ERC12864-10, J2 Terminal Block, J3 ISP/UART, J5 SERVO, Q1 2N7002, Q2 2N7002, SW1 RESET, SW2 ACTION, U1 STM8S[N76E], U2 AMS1117-3.3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

Commit message: updates
Parts:
- J3: footprint MICROJELLY:TRUDEAU_C2X5_SMD -> MICROJELLY:TRUDEAU_C2X5_REG_SMD
- moved C2 3.95 mm to (171.7, 92.5), turned to 90 degrees
- moved C10 3.31 mm to (155.3, 94.5)
- moved R2 2.34 mm to (171.7, 88.7), turned to 90 degrees
- moved J3 2.04 mm to (165.6, 110.0)
- moved BZ1 1.84 mm to (168.0, 100.5)
- moved C6 1.59 mm to (164.7, 94.4), turned to 180 degrees
- moved C5 1.40 mm to (161.9, 98.8)
- moved D1 1.40 mm to (161.9, 102.3)
- moved R5 1.40 mm to (159.8, 100.9)
- moved R4 1.40 mm to (171.7, 83.0), turned to 90 degrees
- moved J1 1.29 mm to (145.6, 89.1)
- moved C9 1.18 mm to (158.9, 98.0)
- moved Q1 1.02 mm to (143.2, 100.6)
- moved Q2 1.02 mm to (147.0, 100.6)
- moved R8 1.02 mm to (136.3, 82.2)
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Routing:
- net GND: track 54.9 -> 70.8 mm, vias 21 -> 16
- net 3V3: track 138.6 -> 146.6 mm
- net SWIM[ICPCK]: track 22.2 -> 27.5 mm
- net BUZZER: track 15.3 -> 18.0 mm
- net RX: track 14.4 -> 16.5 mm
- net TX: track 14.6 -> 16.4 mm
- net LED_RED: track 11.2 -> 9.64 mm
- net LCD_CS: track 23.6 -> 25.1 mm
- net ICPDAT: track 12.9 -> 14.3 mm
- net VIN: track 8.78 -> 7.40 mm
- net SPI_MOSI: track 31.4 -> 30.1 mm
- net T+: track 17.6 -> 16.4 mm
- net LCD_RES: track 23.4 -> 22.3 mm
- net SPI_SCK: track 40.9 -> 39.8 mm
- net Net-(D3-Pad1): track 2.92 -> 3.90 mm
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Other:
- board size 44.9 x 29.9 mm -> 42.9 x 29.9 mm
